File: Schedona gigante/Schedona gigante.kicad_sch (KiCad schematic)
At the start: 0 parts

Commit message: inizio parte di potenza
Parts:
- added U1: (no value), symbol Libreria gigante:STM32H743
Connections:
- new net GND: U1.A1 (VSS_1), U1.A17 (VSS_2), U1.B2 (VSS_3), U1.B6 (VSS_4), U1.C10 (VSS_5), U1.C13 (VSS_6), U1.C16 (VSS_7), U1.F1 (VSS_8), U1.F2 (VSS_9), U1.G10 (VSS_14), U1.G11 (VSS_15), U1.G16 (VSS_16), U1.G2 (VSS_10), U1.G7 (VSS_11), U1.G8 (VSS_12), U1.G9 (VSS_13), U1.H10 (VSS_20), U1.H11 (VSS_21), U1.H7 (VSS_17), U1.H8 (VSS_18), U1.H9 (VSS_19), U1.J10 (VSS_26), U1.J11 (VSS_27), U1.J16 (VSS_28), U1.J17 (VSS_29), U1.J3 (VSS_22), U1.J7 (VSS_23), U1.J8 (VSS_24), U1.J9 (VSS_25), U1.K10 (VSS_33), U1.K11 (VSS_34), U1.K15 (VSS_35), U1.K7 (VSS_30), U1.K8 (VSS_31), U1.K9 (VSS_32), U1.L10 (VSS_39), U1.L11 (VSS_40), U1.L15 (VSS_41), U1.L7 (VSS_36), U1.L8 (VSS_37), U1.L9 (VSS_38), U1.M15 (VSS_42), U1.N16 (VSS_43), U1.P1 (VSSA), U1.R4 (VSS_44), U1.R8 (VSS_45), U1.T12 (VSS_46), U1.U1 (VSS_47), U1.U17 (VSS_48)
- new net VDD_MCU: U1.E11 (VDD_3), U1.E6 (VDD_1), U1.E9 (VDD_2), U1.F5 (VDD_4), U1.G13 (VDD_6), U1.G5 (VDD_5), U1.H5 (VDD_7), U1.J13 (VDD_9), U1.K13 (VDD_11), U1.K5 (VDD_10), U1.L13 (VDD_13), U1.L5 (VDD_12), U1.M13 (VDD_15), U1.M5 (VDD_14), U1.N10 (VDD_18), U1.N11 (VDD_19), U1.N12 (VDD_20), U1.N7 (VDD_16), U1.N8 (VDD_17), U1.P17 (VDD_21)
Other:
- title: (none) -> Power

Commit message: alimentazione pt.2
Parts:
- added C1, C2, C3: 2.2uF, CAPC2012X140N, symbol Libreria gigante:C0805C225K8RAC
- added C10, C11, C12, C13, C14, C5, C6, C7, C8, C9: 100nF, C0402, symbol Libreria gigante:C0402C104K8RAC7411
- added C4: 4.7uF, CAPAE630X800N, symbol Libreria gigante:875105945001
Connections:
- net GND: now also C1.1, C10.2, C11.2, C12.2, C13.2, C14.2, C2.1, C3.1, C4.2, C5.2, C6.2, C7.2, C8.2, C9.2
- net VDD_MCU: now also U1.A6 (VDD_LDO_1), U1.C17 (VDD_LDO_2), U1.H13 (VDD_8), U1.U12 (VDD_LDO_3), C10.1, C11.1, C12.1, C13.1, C14.1, C4.1, C5.1, C6.1, C7.1, C8.1, C9.1
- net at U1.A7 (VCAP_1): now also C1.2
- net at U1.D17 (VCAP_2): now also C2.2
- net at U1.U11 (VCAP_3): now also C3.2
Other:
- note added: "Pulizia alimentazione"
- moved on the sheet: U1B
